File: STM32G071GBU6_breakout.sch (KiCad schematic (older format))
At the start: 14 parts, among them J1 Conn_01x14, J2 Conn_01x14, J3 Conn_01x04, SW1 SW_Push, U1 MCP1700-3302E_SOT23, U2 STM32G071GBU6

Commit message: change SW to KMR2
Parts:
- SW1: footprint Button_Switch_SMD:SW_Push_SPST_NO_Alps_SKRK -> Button_Switch_SMD:SW_Push_1P1T_NO_CK_KMR2
Changed lines of the file:
@@
 F 0 "SW1" V 3554 5198 50  0000 L CNN
 F 1 "SW_Push" V 3645 5198 50  0000 L CNN
-F 2 "Button_Switch_SMD:SW_Push_SPST_NO_Alps_SKRK" H 3600 5250 50  0001 C CNN
+F 2 "Button_Switch_SMD:SW_Push_1P1T_NO_CK_KMR2" H 3600 5250 50  0001 C CNN
 F 3 "~" H 3600 5250 50  0001 C CNN
 	1    3600 5050
